Commit message: 毕设更新

File: agent_project_v2/execution/simulation/models/6061_C_continue/urdf/6061_C_continue.urdf (robot description, URDF)
Before this commit: robot 6061_C_continue, 2 links, 1 joints
Links:
- link Link_1: geometry visual mesh filename=package://6061_C_continue/meshes/Link_1.STL
- link base_link: geometry collision mesh filename=package://6061_C_continue/meshes/base_link.obj; visual mesh filename=package://6061_C_continue/meshes/base_link_new.STL

File: agent_project_v2/execution/simulation/models/calibration_board/urdf/calibration_board.urdf (robot description, URDF)
Before this commit: robot calibration_board, 3 links, 2 joints
Joints:
- joint joint_1: origin xyz=-0.006 0 -0.006 rpy=-1.57 -1.57 0 -> xyz=-0.006 0 -0.006 rpy=-1.5707963267948966 -1.5707963267948966 0
- joint joint_2: origin xyz=-0.0125 0 -0.0125 rpy=-1.57 -1.57 0 -> xyz=-0.0125 0 -0.0125 rpy=-1.5707963267948966 -1.5707963267948966 0
