Commit message: 毕设更新

File: agent_project/simulation/models/jaka_description/urdf/jaka_minicobo_with_rolling_tool_12mm_len248dot37mm.urdf (robot description, URDF)
Before this commit: robot minicobo_v1.4, 12 links, 11 joints
Joints:
- joint joint_RT_1: origin xyz=0.006 0 0.14 rpy=0 0 0 -> xyz=0.006 0 0.24837 rpy=0 0 0
- joint joint_RT_2: origin xyz=-0.006 0 0.14 rpy=0 0 0 -> xyz=-0.006 0 0.24837 rpy=0 0 0
- joint rolling_tool_tcp_joint: origin xyz=0 0 0.14 rpy=0 0 0 -> xyz=0 0 0.24837 rpy=0 0 0
